Commit message: Implemented driver controls and controller manager

File: ezrassor_arm_v2/resource/ezrassor.xacro (robot description, xacro)
@@ -24,5 +24,5 @@
       <origin xyz="0 0 0" rpy=" 0 0 0"/>
       <geometry>
-        <base_unit/>
+        <xacro:base_unit/>
       </geometry>
     </collision>
@@ -30,5 +30,5 @@
       <origin xyz="0 0 0" rpy=" 0 0 0"/>
       <geometry>
-        <base_unit/>
+        <xacro:base_unit/>
       </geometry>
     </visual>
@@ -38,5 +38,5 @@
       <origin xyz="0 0 0" rpy="0 0 0"/>
       <geometry>
-        <robot_wheel />
+        <xacro:robot_wheel />
       </geometry>
       <surface>
@@ -56,5 +56,5 @@
       <origin xyz="0 0 0" rpy="0 0 0"/>
       <geometry>
-        <robot_wheel />
+        <xacro:robot_wheel />
       </geometry>
     </visual>
@@ -62,5 +62,5 @@
       <origin xyz="0 0 0" rpy="0 0 0" />
       <mass value="5"/>
-      <cylinder_inertia m="5" r="0.18" h="0.2"/>
+      <xacro:cylinder_inertia m="5" r="0.18" h="0.2"/>
     </inertial>
   </link>
@@ -69,5 +69,5 @@
       <origin xyz="0 0 0" rpy="0 0 3.14159"/>
       <geometry>
-        <robot_wheel />
+        <xacro:robot_wheel />
       </geometry>
       <surface>
@@ -81,11 +81,11 @@
       <origin xyz="0 0 0" rpy="0 0 3.14159"/>
       <geometry>
-        <robot_wheel />
-      </geometry>
-    </visual>
-    <inertial>
-      <origin xyz="0 0 0" rpy="0 0 3.14159"/>
-      <mass value="5"/>
-      <cylinder_inertia m="5" r="0.18" h="0.2"/>
+        <xacro:robot_wheel />
+      </geometry>
+    </visual>
+    <inertial>
+      <origin xyz="0 0 0" rpy="0 0 3.14159"/>
+      <mass value="5"/>
+      <xacro:cylinder_inertia m="5" r="0.18" h="0.2"/>
     </inertial>
   </link>
@@ -94,5 +94,5 @@
       <origin xyz="0 0 0" rpy="0 0 0"/>
       <geometry>
-        <robot_wheel />
+        <xacro:robot_wheel />
       </geometry>
         <surface>
@@ -106,11 +106,11 @@
       <origin xyz="0 0 0" rpy="0 0 0"/>
       <geometry>
-        <robot_wheel />
-      </geometry>
-    </visual>
-    <inertial>
-      <origin xyz="0 0 0" rpy="0 0 0"/>
-      <mass value="5"/>
-      <cylinder_inertia m="5" r="0.18" h="0.2"/>
+        <xacro:robot_wheel />
+      </geometry>
+    </visual>
+    <inertial>
+      <origin xyz="0 0 0" rpy="0 0 0"/>
+      <mass value="5"/>
+      <xacro:cylinder_inertia m="5" r="0.18" h="0.2"/>
     </inertial>
   </link>
@@ -119,5 +119,5 @@
       <origin xyz="0 0 0" rpy="0 0 3.14159"/>
       <geometry>
-        <robot_wheel />
+        <xacro:robot_wheel />
       </geometry>
       <surface>
@@ -131,11 +131,11 @@
       <origin xyz="0 0 0" rpy="0 0 3.14159"/>
       <geometry>
-        <robot_wheel />
-      </geometry>
-    </visual>
-    <inertial>
-      <origin xyz="0 0 0" rpy="0 0 3.14159"/>
-      <mass value="5"/>
-      <cylinder_inertia m="5" r="0.18" h="0.2"/>
+        <xacro:robot_wheel />
+      </geometry>
+    </visual>
+    <inertial>
+      <origin xyz="0 0 0" rpy="0 0 3.14159"/>
+      <mass value="5"/>
+      <xacro:cylinder_inertia m="5" r="0.18" h="0.2"/>
     </inertial>
   </link>
@@ -144,5 +144,5 @@
       <origin xyz="0 0 0" rpy="0 0 0"/>
       <geometry>
-        <drum_arm />
+        <xacro:drum_arm />
       </geometry>
     </collision>
@@ -150,11 +150,11 @@
       <origin xyz="0 0 0" rpy="0 0 0" />
       <geometry>
-        <drum_arm />
-      </geometry>
-    </visual>
-    <inertial>
-      <origin xyz="0 0 0" rpy="0 0 0"/>
-      <mass value="5"/>
-      <cylinder_inertia m="5" r="0.05" h="0.3"/>
+        <xacro:drum_arm />
+      </geometry>
+    </visual>
+    <inertial>
+      <origin xyz="0 0 0" rpy="0 0 0"/>
+      <mass value="5"/>
+      <xacro:cylinder_inertia m="5" r="0.05" h="0.3"/>
     </inertial>
   </link>
@@ -163,5 +163,5 @@
       <origin xyz="0 0 0" rpy="3.1415 0 3.1415"/>
       <geometry>
-        <drum_arm />
+        <xacro:drum_arm />
       </geometry>
     </collision>
@@ -169,5 +169,5 @@
       <origin xyz="0 0 0" rpy="3.1415 0 3.1415"/>
       <geometry>
-        <drum_arm />
+        <xacro:drum_arm />
       </geometry>
     </visual>
@@ -175,5 +175,5 @@
       <origin xyz="0 0 0" rpy="0 0 3.1415"/>
       <mass value="5"/>
-      <cylinder_inertia m="5" r="0.05" h="0.3"/>
+      <xacro:cylinder_inertia m="5" r="0.05" h="0.3"/>
       <inertia
         ixx="1.0" ixy="0.0" ixz="0.0"
@@ -198,11 +198,11 @@
       <origin xyz="0 0 0" rpy="0 0 0"/>
       <geometry>
-        <robot_arm_drum />
-      </geometry>
-    </visual>
-    <inertial>
-      <origin xyz="0 0 0" rpy="0 0 0"/>
-      <mass value="5"/>
-      <cylinder_inertia m="5" r="0.1839" h="1.0"/>
+        <xacro:robot_arm_drum />
+      </geometry>
+    </visual>
+    <inertial>
+      <origin xyz="0 0 0" rpy="0 0 0"/>
+      <mass value="5"/>
+      <xacro:cylinder_inertia m="5" r="0.1839" h="1.0"/>
     </inertial>
   </link>
@@ -223,14 +223,15 @@
       <origin xyz="0 0 0" rpy="3.1415 0 3.14159"/>
       <geometry>
-        <robot_arm_drum />
-      </geometry>
-    </visual>
-    <inertial>
-      <origin xyz="0 0 0" rpy="0 0 3.14159"/>
-      <mass value="5"/>
-      <cylinder_inertia m="5" r="0.1839" h="1.0"/>
+        <xacro:robot_arm_drum />
+      </geometry>
+    </visual>
+    <inertial>
+      <origin xyz="0 0 0" rpy="0 0 3.14159"/>
+      <mass value="5"/>
+      <xacro:cylinder_inertia m="5" r="0.1839" h="1.0"/>
     </inertial>
   </link>
   <!-- Transmissions -->
+  <!--
   <transmission name="left_wheel_front_tran">
     <type>transmission_interface/SimpleTransmission</type>
@@ -313,4 +314,5 @@
     </actuator>
   </transmission>
+  -->
   <!-- Front Camera Added -->
   <link name="depth_camera_front">
@@ -331,5 +333,5 @@
       <mass value="${cameraMass}" />
       <origin xyz="0 0 0" rpy="0 0 0"/>
-      <box_inertia m="${cameraMass}" x="${cameraSize}" y="${cameraSize}" z="${cameraSize}" />
+      <xacro:box_inertia m="${cameraMass}" x="${cameraSize}" y="${cameraSize}" z="${cameraSize}" />
       <inertia ixx="1e-6" ixy="0" ixz="0" iyy="1e-6" iyz="0" izz="1e-6" />
     </inertial>
@@ -352,5 +354,5 @@
       <mass value="${cameraMass}" />
       <origin xyz="0 0 0" rpy="0 0 0"/>
-      <box_inertia m="${cameraMass}" x="${cameraSize}" y="${cameraSize}" z="${cameraSize}" />
+      <xacro:box_inertia m="${cameraMass}" x="${cameraSize}" y="${cameraSize}" z="${cameraSize}" />
       <inertia ixx="1e-6" ixy="0" ixz="0" iyy="1e-6" iyz="0" izz="1e-6" />
     </inertial>
@@ -444,3 +446,77 @@
     <joint_properties damping="0.0" friction="0.0"/>
   </joint>
+  <ros2_control name="GazeboSystem" type="system">
+            <hardware>
+                <plugin>gazebo_ros2_control/GazeboSystem</plugin>
+            </hardware>
+            <joint name="left_wheel_front_joint">
+            <command_interface name="velocity">
+                <param name="min">-10</param>
+                <param name="max">10</param>
+            </command_interface>
+            <state_interface name="position" />
+            <state_interface name="velocity" />
+        </joint>
+        <joint name="left_wheel_back_joint">
+            <command_interface name="velocity">
+                <param name="min">-10</param>
+                <param name="max">10</param>
+            </command_interface>
+            <state_interface name="position" />
+            <state_interface name="velocity" />
+        </joint>
+        <joint name="right_wheel_front_joint">
+            <command_interface name="velocity">
+                <param name="min">-10</param>
+                <param name="max">10</param>
+            </command_interface>
+            <state_interface name="position" />
+            <state_interface name="velocity" />
+        </joint>
+        <joint name="right_wheel_back_joint">
+            <command_interface name="velocity">
+                <param name="min">-10</param>
+                <param name="max">10</param>
+            </command_interface>
+            <state_interface name="position" />
+            <state_interface name="velocity" />
+        </joint>
+        <joint name="arm_back_joint">
+            <command_interface name="velocity">
+                <param name="min">-10</param>
+                <param name="max">10</param>
+            </command_interface>
+            <state_interface name="position" />
+            <state_interface name="velocity" />
+        </joint>
+        <joint name="drum_back_joint">
+            <command_interface name="velocity">
+                <param name="min">-10</param>
+                <param name="max">10</param>
+            </command_interface>
+            <state_interface name="position" />
+            <state_interface name="velocity" />
+        </joint>
+        <joint name="arm_front_joint">
+            <command_interface name="velocity">
+                <param name="min">-10</param>
+                <param name="max">10</param>
+            </command_interface>
+            <state_interface name="position" />
+            <state_interface name="velocity" />
+        </joint>
+        <joint name="drum_front_joint">
+            <command_interface name="velocity">
+                <param name="min">-10</param>
+                <param name="max">10</param>
+            </command_interface>
+            <state_interface name="position" />
+            <state_interface name="velocity" />
+        </joint>
+        </ros2_control>
+  <gazebo>
+    <plugin filename="libgazebo_ros2_control.so" name="gazebo_ros2_control">
+      <parameters>$(find ezrassor_arm_v2)/config/paver_arm_rover/default_position_controllers.yaml</parameters>
+    </plugin>
+  </gazebo>
 </robot>

File: ezrassor_arm_v2/resource/ezrassor_arm_v2.xacro (robot description, xacro)
@@ -24,5 +24,5 @@
       <origin xyz="0 0 0" rpy=" 0 0 0"/>
       <geometry>
-        <base_unit/>
+        <xacro:base_unit/>
       </geometry>
     </collision>
@@ -30,5 +30,5 @@
       <origin xyz="0 0 0" rpy=" 0 0 0"/>
       <geometry>
-        <base_unit/>
+        <xacro:base_unit/>
       </geometry>
     </visual>
@@ -38,5 +38,5 @@
       <origin xyz="0 0 0" rpy="0 0 0"/>
       <geometry>
-        <robot_wheel />
+        <xacro:robot_wheel />
       </geometry>
       <surface>
@@ -56,5 +56,5 @@
       <origin xyz="0 0 0" rpy="0 0 0"/>
       <geometry>
-        <robot_wheel />
+        <xacro:robot_wheel />
       </geometry>
     </visual>
@@ -62,5 +62,5 @@
       <origin xyz="0 0 0" rpy="0 0 0" />
       <mass value="5"/>
-      <cylinder_inertia m="5" r="0.18" h="0.2"/>
+      <xacro:cylinder_inertia m="5" r="0.18" h="0.2"/>
     </inertial>
   </link>
@@ -69,5 +69,5 @@
       <origin xyz="0 0 0" rpy="0 0 3.14159"/>
       <geometry>
-        <robot_wheel />
+        <xacro:robot_wheel />
       </geometry>
       <surface>
@@ -81,5 +81,5 @@
       <origin xyz="0 0 0" rpy="0 0 3.14159"/>
       <geometry>
-        <robot_wheel />
+        <xacro:robot_wheel />
       </geometry>
     </visual>
@@ -87,5 +87,5 @@
       <origin xyz="0 0 0" rpy="0 0 3.14159"/>
       <mass value="5"/>
-      <cylinder_inertia m="5" r="0.18" h="0.2"/>
+      <xacro:cylinder_inertia m="5" r="0.18" h="0.2"/>
     </inertial>
   </link>
@@ -94,5 +94,5 @@
       <origin xyz="0 0 0" rpy="0 0 0"/>
       <geometry>
-        <robot_wheel />
+        <xacro:robot_wheel />
       </geometry>
         <surface>
@@ -106,5 +106,5 @@
       <origin xyz="0 0 0" rpy="0 0 0"/>
       <geometry>
-        <robot_wheel />
+        <xacro:robot_wheel />
       </geometry>
     </visual>
@@ -112,5 +112,5 @@
       <origin xyz="0 0 0" rpy="0 0 0"/>
       <mass value="5"/>
-      <cylinder_inertia m="5" r="0.18" h="0.2"/>
+      <xacro:cylinder_inertia m="5" r="0.18" h="0.2"/>
     </inertial>
   </link>
@@ -119,5 +119,5 @@
       <origin xyz="0 0 0" rpy="0 0 3.14159"/>
       <geometry>
-        <robot_wheel />
+        <xacro:robot_wheel />
       </geometry>
       <surface>
@@ -131,5 +131,5 @@
       <origin xyz="0 0 0" rpy="0 0 3.14159"/>
       <geometry>
-        <robot_wheel />
+        <xacro:robot_wheel />
       </geometry>
     </visual>
@@ -137,5 +137,5 @@
       <origin xyz="0 0 0" rpy="0 0 3.14159"/>
       <mass value="5"/>
-      <cylinder_inertia m="5" r="0.18" h="0.2"/>
+      <xacro:cylinder_inertia m="5" r="0.18" h="0.2"/>
     </inertial>
   </link>
@@ -144,5 +144,5 @@
       <origin xyz="0 0 0" rpy="3.1415 0 3.1415"/>
       <geometry>
-        <drum_arm />
+        <xacro:drum_arm />
       </geometry>
     </collision>
@@ -150,5 +150,5 @@
       <origin xyz="0 0 0" rpy="3.1415 0 3.1415"/>
       <geometry>
-        <drum_arm />
+        <xacro:drum_arm />
       </geometry>
     </visual>
@@ -156,5 +156,5 @@
       <origin xyz="0 0 0" rpy="0 0 3.1415"/>
       <mass value="5"/>
-      <cylinder_inertia m="5" r="0.05" h="0.3"/>
+      <xacro:cylinder_inertia m="5" r="0.05" h="0.3"/>
       <inertia
         ixx="1.0" ixy="0.0" ixz="0.0"
@@ -179,5 +179,5 @@
       <origin xyz="0 0 0" rpy="3.1415 0 3.14159"/>
       <geometry>
-        <robot_arm_drum />
+        <xacro:robot_arm_drum/>
       </geometry>
     </visual>
@@ -185,5 +185,5 @@
       <origin xyz="0 0 0" rpy="0 0 3.14159"/>
       <mass value="5"/>
-      <cylinder_inertia m="5" r="0.1839" h="1.0"/>
+      <xacro:cylinder_inertia m="5" r="0.1839" h="1.0"/>
     </inertial>
   </link>
@@ -203,5 +203,5 @@
       <origin xyz="0 0 0" rpy=" 0 0 0"/>
       <geometry>
-        <link1/>
+        <xacro:link1/>
       </geometry>
     </collision>
@@ -209,5 +209,5 @@
       <origin xyz="0 0 0" rpy=" 0 0 0"/>
       <geometry>
-        <link1/>
+        <xacro:link1/>
       </geometry>
     </visual>
@@ -227,5 +227,5 @@
       <origin xyz="0 0.08 0.135" rpy=" 0 0 0"/>
       <geometry>
-        <link2/>
+        <xacro:link2/>
       </geometry>
     </collision>
@@ -233,5 +233,5 @@
       <origin xyz="0 0.08 0.135" rpy=" 0 0 0"/>
       <geometry>
-        <link2/>
+        <xacro:link2/>
       </geometry>
     </visual>
@@ -251,5 +251,5 @@
       <origin xyz="0.25 0.1 0" rpy=" 0 0 0"/>
       <geometry>
-        <link3/>
+        <xacro:link3/>
       </geometry>
     </collision>
@@ -257,5 +257,5 @@
       <origin xyz="0.25 0.1 0" rpy=" 0 0 0"/>
       <geometry>
-        <link3/>
+        <xacro:link3/>
       </geometry>
     </visual>
@@ -275,5 +275,5 @@
       <origin xyz="0.23 0 0" rpy=" 0 0 0"/>
       <geometry>
-        <link4/>
+        <xacro:link4/>
       </geometry>
     </collision>
@@ -281,5 +281,5 @@
       <origin xyz="0.23 0 0" rpy=" 0 0 0"/>
       <geometry>
-        <link4/>
+        <xacro:link4/>
       </geometry>
     </visual>
@@ -299,5 +299,5 @@
       <origin xyz="0 0.12 0" rpy=" 0 0 0"/>
       <geometry>
-        <link5/>
+        <xacro:link5/>
       </geometry>
     </collision>
@@ -305,5 +305,5 @@
       <origin xyz="0 0.12 0" rpy=" 0 0 0"/>
       <geometry>
-        <link5/>
+        <xacro:link5/>
       </geometry>
     </visual>
@@ -323,5 +323,5 @@
       <origin xyz="0.096 0 -0.24" rpy=" 0 0 0"/>
       <geometry>
-        <link6/>
+        <xacro:link6/>
       </geometry>
     </collision>
@@ -329,5 +329,5 @@
       <origin xyz="0.096 0 -0.24" rpy=" 0 0 0"/>
       <geometry>
-        <link6/>
+        <xacro:link6/>
       </geometry>
     </visual>
@@ -347,5 +347,5 @@
       <origin xyz="0.04 0.0 -0.04" rpy=" 0 0 0"/>
       <geometry>
-        <arm_camera/>
+        <xacro:arm_camera/>
       </geometry>
     </visual>
@@ -365,5 +365,5 @@
       <origin xyz="0 0 0" rpy=" 0 0 0"/>
       <geometry>
-        <grabber1/>
+        <xacro:grabber1/>
       </geometry>
       <contact_coefficients>
@@ -388,5 +388,5 @@
       <origin xyz="0 0 0" rpy=" 0 0 0"/>
       <geometry>
-        <grabber1/>
+        <xacro:grabber1/>
       </geometry>
     </visual>
@@ -406,5 +406,5 @@
       <origin xyz="0 0 0" rpy=" 0 0 0"/>
       <geometry>
-        <grabber2/>
+        <xacro:grabber2/>
       </geometry>
       <contact_coefficients>
@@ -429,5 +429,5 @@
       <origin xyz="0 0 0" rpy=" 0 0 0"/>
       <geometry>
-        <grabber2/>
+        <xacro:grabber2/>
       </geometry>
     </visual>
@@ -447,5 +447,5 @@
       <origin xyz="0.2 0 0" rpy=" 0 -0.60 0"/>
       <geometry>
-        <drum_arm/>
+        <xacro:drum_arm/>
       </geometry>
     </visual>
@@ -474,9 +474,10 @@
       <origin xyz="0.1 0.06 0.1" rpy=" 0 0 0"/>
       <geometry>
-        <platform/>
+        <xacro:platform/>
       </geometry>
     </visual>
   </link>
   <!-- Transmissions -->
+  <!--
   <transmission name="left_wheel_front_tran">
     <type>transmission_interface/SimpleTransmission</type>
@@ -609,4 +610,5 @@
     </actuator>
   </transmission>
+  -->
   <!-- Front Camera Added -->
   <link name="depth_camera_front">
@@ -627,5 +629,5 @@
       <mass value="${cameraMass}" />
       <origin xyz="0 0 0" rpy="0 0 0"/>
-      <box_inertia m="${cameraMass}" x="${cameraSize}" y="${cameraSize}" z="${cameraSize}" />
+      <xacro:box_inertia m="${cameraMass}" x="${cameraSize}" y="${cameraSize}" z="${cameraSize}" />
       <inertia ixx="1e-6" ixy="0" ixz="0" iyy="1e-6" iyz="0" izz="1e-6" />
     </inertial>
@@ -648,5 +650,5 @@
       <mass value="${cameraMass}" />
       <origin xyz="0 0 0" rpy="0 0 0"/>
-      <box_inertia m="${cameraMass}" x="${cameraSize}" y="${cameraSize}" z="${cameraSize}" />
+      <xacro:box_inertia m="${cameraMass}" x="${cameraSize}" y="${cameraSize}" z="${cameraSize}" />
       <inertia ixx="1e-6" ixy="0" ixz="0" iyy="1e-6" iyz="0" izz="1e-6" />
     </inertial>
@@ -676,5 +678,5 @@
   </joint>
   <link name="depth_camera_optical_frame"/>
-  <joint type="continuous" name="left_wheel_front_hinge">
+  <joint type="continuous" name="left_wheel_front_joint">
     <origin xyz="0.20 0.285 0" rpy="0 0 0"/>
     <child link="left_wheel_front"/>
@@ -684,5 +686,5 @@
     <joint_properties damping="0.0" friction="0.0"/>
   </joint>
-  <joint type="continuous" name="right_wheel_front_hinge">
+  <joint type="continuous" name="right_wheel_front_joint">
     <origin xyz="0.20 -0.285 0" rpy="0 0 0"/>
     <child link="right_wheel_front"/>
@@ -692,5 +694,5 @@
     <joint_properties damping="0.0" friction="0.0"/>
   </joint>
-  <joint type="continuous" name="left_wheel_back_hinge">
+  <joint type="continuous" name="left_wheel_back_joint">
     <origin xyz="-0.20 0.285 0" rpy="0 0 0"/>
     <child link="left_wheel_back"/>
@@ -700,5 +702,5 @@
     <joint_properties damping="0.0" friction="0.0"/>
   </joint>
-  <joint type="continuous" name="right_wheel_back_hinge">
+  <joint type="continuous" name="right_wheel_back_joint">
     <origin xyz="-0.20 -0.285 0" rpy="0 0 0"/>
     <child link="right_wheel_back"/>
@@ -708,5 +710,5 @@
     <joint_properties damping="0.0" friction="0.0"/>
   </joint>
-  <joint type="continuous" name="arm_back_hinge">
+  <joint type="continuous" name="arm_back_joint">
     <origin xyz="-0.20 0 0" rpy="0 0 0"/>
     <child link="arm_back"/>
@@ -716,5 +718,5 @@
     <joint_properties damping="0.0" friction="0.0"/>
   </joint>
-  <joint type="continuous" name="drum_back_hinge">
+  <joint type="continuous" name="drum_back_joint">
     <origin xyz="-0.388245 0 0" rpy="3.1415 0 0"/>
     <child link="drum_back"/>
@@ -800,11 +802,130 @@
     <limit lower="-0.02" upper="0.0225" effort="10" velocity="0.005"/>
   </joint>
-  <ros2_control_arm_joint1/>
-  <ros2_control_arm_joint2/>
-  <ros2_control_arm_joint3/>
-  <ros2_control_arm_joint4/>
-  <ros2_control_arm_joint5/>
-  <ros2_control_arm_grabber1/>
-  <ros2_control_arm_grabber2/>
+  <ros2_control name="GazeboSystem" type="system">
+            <hardware>
+                <plugin>gazebo_ros2_control/GazeboSystem</plugin>
+            </hardware>
+            <joint name="joint1">
+                <command_interface name="position">
+                    <param name="min">-15</param>
+                    <param name="max">15</param>
+                </command_interface>
+                <state_interface name="position">
+                    <param name="initial_value">1.0</param>
+                </state_interface>
+                <state_interface name="velocity"/>
+                <state_interface name="effort"/>
+            </joint>
+            <joint name="joint2">
+                <command_interface name="position">
+                    <param name="min">-15</param>
+                    <param name="max">15</param>
+                </command_interface>
+                <state_interface name="position">
+                    <param name="initial_value">1.0</param>
+                </state_interface>
+                <state_interface name="velocity"/>
+                <state_interface name="effort"/>
+            </joint>
+            <joint name="joint3">
+                <command_interface name="position">
+                    <param name="min">-15</param>
+                    <param name="max">15</param>
+                </command_interface>
+                <state_interface name="position">
+                    <param name="initial_value">1.0</param>
+                </state_interface>
+                <state_interface name="velocity"/>
+                <state_interface name="effort"/>
+            </joint>
+            <joint name="joint4">
+                <command_interface name="position">
+                    <param name="min">-15</param>
+                    <param name="max">15</param>
+                </command_interface>
+                <state_interface name="position">
+                    <param name="initial_value">1.0</param>
+                </state_interface>
+                <state_interface name="velocity"/>
+                <state_interface name="effort"/>
+            </joint>
+            <joint name="joint5">
+                <command_interface name="position">
+                    <param name="min">-15</param>
+                    <param name="max">15</param>
+                </command_interface>
+                <state_interface name="position">
+                    <param name="initial_value">1.0</param>
+                </state_interface>
+                <state_interface name="velocity"/>
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