Commit message: Ros Controls now load based on the rover type

File: ezrassor_arm_v2/resource/ezrassor.xacro (robot description, xacro)
@@ -382,5 +382,5 @@
   </joint>
   <link name="depth_camera_optical_frame"/>
-  <joint type="continuous" name="left_wheel_front_hinge">
+  <joint type="continuous" name="left_wheel_front_joint">
     <origin xyz="0.20 0.285 0" rpy="0 0 0"/>
     <child link="left_wheel_front"/>
@@ -390,5 +390,5 @@
     <joint_properties damping="0.0" friction="0.0"/>
   </joint>
-  <joint type="continuous" name="right_wheel_front_hinge">
+  <joint type="continuous" name="right_wheel_front_joint">
     <origin xyz="0.20 -0.285 0" rpy="0 0 0"/>
     <child link="right_wheel_front"/>
@@ -398,5 +398,5 @@
     <joint_properties damping="0.0" friction="0.0"/>
   </joint>
-  <joint type="continuous" name="left_wheel_back_hinge">
+  <joint type="continuous" name="left_wheel_back_joint">
     <origin xyz="-0.20 0.285 0" rpy="0 0 0"/>
     <child link="left_wheel_back"/>
@@ -406,5 +406,5 @@
     <joint_properties damping="0.0" friction="0.0"/>
   </joint>
-  <joint type="continuous" name="right_wheel_back_hinge">
+  <joint type="continuous" name="right_wheel_back_joint">
     <origin xyz="-0.20 -0.285 0" rpy="0 0 0"/>
     <child link="right_wheel_back"/>
@@ -414,5 +414,5 @@
     <joint_properties damping="0.0" friction="0.0"/>
   </joint>
-  <joint type="continuous" name="arm_front_hinge">
+  <joint type="continuous" name="arm_front_joint">
     <origin xyz="0.20 0 0" rpy="3.1415 0 0"/>
     <child link="arm_front"/>
@@ -422,5 +422,5 @@
     <joint_properties damping="0.0" friction="0.0"/>
   </joint>
-  <joint type="continuous" name="arm_back_hinge">
+  <joint type="continuous" name="arm_back_joint">
     <origin xyz="-0.20 0 0" rpy="0 0 0"/>
     <child link="arm_back"/>
@@ -430,5 +430,5 @@
     <joint_properties damping="0.0" friction="0.0"/>
   </joint>
-  <joint type="continuous" name="drum_front_hinge">
+  <joint type="continuous" name="drum_front_joint">
     <origin xyz="0.388245 0 0" rpy="3.1415 0 0"/>
     <child link="drum_front"/>
@@ -438,5 +438,5 @@
     <joint_properties damping="0.0" friction="0.0"/>
   </joint>
-  <joint type="continuous" name="drum_back_hinge">
+  <joint type="continuous" name="drum_back_joint">
     <origin xyz="-0.388245 0 0" rpy="3.1415 0 0"/>
     <child link="drum_back"/>
