Commit message: fixed moveit controller yaml, add moveit interface

File: ezrassor_arm_v2/resource/arm_model.urdf (robot description, URDF)
Before this commit: robot ezrassor, 22 links, 21 joints
Links:
- link arm_back: geometry collision mesh filename=package://ezrassor_arm_v2/meshes/drum_arm.dae scale=0.35 0.35 0.35; visual mesh filename=package://ezrassor_arm_v2/meshes/drum_arm.dae scale=0.35 0.35 0.35
- link arm_camera: geometry collision mesh filename=package://ezrassor_arm_v2/meshes/arm_camera.dae scale=0.35 0.35 0.35; visual mesh filename=package://ezrassor_arm_v2/meshes/arm_camera.dae scale=0.35 0.35 0.35
- link arm_front: geometry collision mesh filename=package://ezrassor_arm_v2/meshes/drum_arm.dae scale=0.35 0.35 0.35; visual mesh filename=package://ezrassor_arm_v2/meshes/drum_arm.dae scale=0.35 0.35 0.35
- link body: geometry collision mesh filename=package://ezrassor_arm_v2/meshes/base_unit.dae scale=0.35 0.35 0.35; visual mesh filename=package://ezrassor_arm_v2/meshes/base_unit.dae scale=0.35 0.35 0.35
- link drum_back: geometry collision cylinder length=1.0 radius=0.1839; visual mesh filename=package://ezrassor_arm_v2/meshes/drum.dae scale=0.35 0.35 0.35
- link grabber1: geometry collision mesh filename=package://ezrassor_arm_v2/meshes/grabber1.dae scale=0.35 0.35 0.35; visual mesh filename=package://ezrassor_arm_v2/meshes/grabber1.dae scale=0.35 0.35 0.35
- link grabber2: geometry collision mesh filename=package://ezrassor_arm_v2/meshes/grabber2.dae scale=0.35 0.35 0.35; visual mesh filename=package://ezrassor_arm_v2/meshes/grabber2.dae scale=0.35 0.35 0.35
- link left_wheel_back: geometry collision mesh filename=package://ezrassor_arm_v2/meshes/wheel.dae scale=0.35 0.35 0.35; visual mesh filename=package://ezrassor_arm_v2/meshes/wheel.dae scale=0.35 0.35 0.35
- link left_wheel_front: geometry collision mesh filename=package://ezrassor_arm_v2/meshes/wheel.dae scale=0.35 0.35 0.35; visual mesh filename=package://ezrassor_arm_v2/meshes/wheel.dae scale=0.35 0.35 0.35
- link link1: geometry collision mesh filename=package://ezrassor_arm_v2/meshes/link1.dae scale=0.35 0.35 0.35; visual mesh filename=package://ezrassor_arm_v2/meshes/link1.dae scale=0.35 0.35 0.35
- link link2: geometry collision mesh filename=package://ezrassor_arm_v2/meshes/link2.dae scale=0.35 0.35 0.35; visual mesh filename=package://ezrassor_arm_v2/meshes/link2.dae scale=0.35 0.35 0.35
- link link3: geometry collision mesh filename=package://ezrassor_arm_v2/meshes/link3.dae scale=0.35 0.35 0.35; visual mesh filename=package://ezrassor_arm_v2/meshes/link3.dae scale=0.35 0.35 0.35
- link link4: geometry collision mesh filename=package://ezrassor_arm_v2/meshes/link4.dae scale=0.35 0.35 0.35; visual mesh filename=package://ezrassor_arm_v2/meshes/link4.dae scale=0.35 0.35 0.35
- link link5: geometry collision mesh filename=package://ezrassor_arm_v2/meshes/link5.dae scale=0.35 0.35 0.35; visual mesh filename=package://ezrassor_arm_v2/meshes/link5.dae scale=0.35 0.35 0.35
- link link6: geometry collision mesh filename=package://ezrassor_arm_v2/meshes/link6.1.dae scale=0.35 0.35 0.45; visual mesh filename=package://ezrassor_arm_v2/meshes/link6.1.dae scale=0.35 0.35 0.45
- link platform: geometry collision mesh filename=package://ezrassor_arm_v2/meshes/platform.dae scale=2 2 2; visual mesh filename=package://ezrassor_arm_v2/meshes/platform.dae scale=2 2 2
- link right_wheel_back: geometry collision mesh filename=package://ezrassor_arm_v2/meshes/wheel.dae scale=0.35 0.35 0.35; visual mesh filename=package://ezrassor_arm_v2/meshes/wheel.dae scale=0.35 0.35 0.35
- link right_wheel_front: geometry collision mesh filename=package://ezrassor_arm_v2/meshes/wheel.dae scale=0.35 0.35 0.35; visual mesh filename=package://ezrassor_arm_v2/meshes/wheel.dae scale=0.35 0.35 0.35

Commit message: added arm command msg, topic fix and sim physics

File: ezrassor_arm_v2/resource/arm_model.urdf (robot description, URDF)
Before this commit: robot ezrassor, 22 links, 21 joints
Joints:
- removed joint arm_back_hinge
- removed joint drum_back_hinge
- removed joint left_wheel_back_hinge
- removed joint left_wheel_front_hinge
- removed joint right_wheel_back_hinge
- removed joint right_wheel_front_hinge
- added joint arm_back_joint: type continuous, parent base_link, child arm_back, origin xyz=-0.20 0 0 rpy=0 0 0, axis 0 1 0, limit effort=100 velocity=100
- added joint drum_back_joint: type continuous, parent arm_back, child drum_back, origin xyz=-0.388245 0 0 rpy=3.1415 0 0, axis 0 1 0, limit effort=100 velocity=100
- added joint left_wheel_back_joint: type continuous, parent base_link, child left_wheel_back, origin xyz=-0.20 0.285 0 rpy=0 0 0, axis 0 1 0, limit effort=100 velocity=100
- added joint left_wheel_front_joint: type continuous, parent base_link, child left_wheel_front, origin xyz=0.20 0.285 0 rpy=0 0 0, axis 0 1 0, limit effort=100 velocity=100
- added joint right_wheel_back_joint: type continuous, parent base_link, child right_wheel_back, origin xyz=-0.20 -0.285 0 rpy=0 0 0, axis 0 1 0, limit effort=100 velocity=100
- added joint right_wheel_front_joint: type continuous, parent base_link, child right_wheel_front, origin xyz=0.20 -0.285 0 rpy=0 0 0, axis 0 1 0, limit effort=100 velocity=100

File: ezrassor_arm_v2/resource/ezrassor_arm_v2.xacro (robot description, xacro)
@@ -479,8 +479,7 @@
   </link>
   <!-- Transmissions -->
-  <!--
   <transmission name="left_wheel_front_tran">
     <type>transmission_interface/SimpleTransmission</type>
-    <joint name="left_wheel_front_hinge">
+    <joint name="left_wheel_front_joint">
       <hardwareInterface>hardware_interface/VelocityJointInterface</hardwareInterface>
     </joint>
@@ -492,5 +491,5 @@
   <transmission name="left_wheel_back_tran">
     <type>transmission_interface/SimpleTransmission</type>
-    <joint name="left_wheel_back_hinge">
+    <joint name="left_wheel_back_joint">
       <hardwareInterface>hardware_interface/VelocityJointInterface</hardwareInterface>
     </joint>
@@ -502,5 +501,5 @@
   <transmission name="right_wheel_front_tran">
     <type>transmission_interface/SimpleTransmission</type>
-    <joint name="right_wheel_front_hinge">
+    <joint name="right_wheel_front_joint">
       <hardwareInterface>hardware_interface/VelocityJointInterface</hardwareInterface>
     </joint>
@@ -512,5 +511,5 @@
   <transmission name="right_wheel_back_tran">
     <type>transmission_interface/SimpleTransmission</type>
-    <joint name="right_wheel_back_hinge">
+    <joint name="right_wheel_back_joint">
       <hardwareInterface>hardware_interface/VelocityJointInterface</hardwareInterface>
     </joint>
@@ -522,5 +521,5 @@
   <transmission name="arm_back_tran">
     <type>transmission_interface/SimpleTransmission</type>
-    <joint name="arm_back_hinge">
+    <joint name="arm_back_joint">
       <hardwareInterface>hardware_interface/VelocityJointInterface</hardwareInterface>
     </joint>
@@ -530,10 +529,10 @@
     </actuator>
   </transmission>
-  <transmission name="drum_back_hinge_tran">
-    <type>transmission_interface/SimpleTransmission</type>
-    <joint name="drum_back_hinge">
-      <hardwareInterface>hardware_interface/VelocityJointInterface</hardwareInterface>
-    </joint>
-    <actuator name="drum_back_hinge_motor">
+  <transmission name="drum_back_joint_tran">
+    <type>transmission_interface/SimpleTransmission</type>
+    <joint name="drum_back_joint">
+      <hardwareInterface>hardware_interface/VelocityJointInterface</hardwareInterface>
+    </joint>
+    <actuator name="drum_back_joint_motor">
       <hardwareInterface>hardware_interface/VelocityJointInterface</hardwareInterface>
       <mechanicalReduction>1</mechanicalReduction>
@@ -813,5 +812,5 @@
                 </command_interface>
                 <state_interface name="position">
-                    <param name="initial_value">1.0</param>
+                    <param name="initial_value">0.0</param>
                 </state_interface>
                 <state_interface name="velocity"/>
@@ -824,5 +823,5 @@
                 </command_interface>
                 <state_interface name="position">
-                    <param name="initial_value">1.0</param>
+                    <param name="initial_value">0.0</param>
                 </state_interface>
                 <state_interface name="velocity"/>
@@ -835,5 +834,5 @@
                 </command_interface>
                 <state_interface name="position">
-                    <param name="initial_value">1.0</param>
+                    <param name="initial_value">0.0</param>
                 </state_interface>
                 <state_interface name="velocity"/>
@@ -846,5 +845,5 @@
                 </command_interface>
                 <state_interface name="position">
-                    <param name="initial_value">1.0</param>
+                    <param name="initial_value">0.0</param>
                 </state_interface>
                 <state_interface name="velocity"/>
@@ -857,5 +856,5 @@
                 </command_interface>
                 <state_interface name="position">
-                    <param name="initial_value">1.0</param>
+                    <param name="initial_value">0.0</param>
                 </state_interface>
                 <state_interface name="velocity"/>
