Commit message: gazebo_ros2_control integration started

File: ezrassor_arm_v2/resource/ezrassor_arm_v2.xacro (robot description, xacro)
@@ -800,3 +800,15 @@
     <limit lower="-0.02" upper="0.0225" effort="10" velocity="0.005"/>
   </joint>
+  <ros2_control_arm_joint1/>
+  <ros2_control_arm_joint2/>
+  <ros2_control_arm_joint3/>
+  <ros2_control_arm_joint4/>
+  <ros2_control_arm_joint5/>
+  <ros2_control_arm_grabber1/>
+  <ros2_control_arm_grabber2/>
+  <gazebo>
+    <plugin filename="libgazebo_ros2_control.so" name="gazebo_ros2_control">
+      <parameters>$(find ezrassor_arm_v2)/config/paver_arm_rover/default_position_controllers.yaml</parameters>
+    </plugin>
+  </gazebo>
 </robot>

File: ezrassor_arm_v2/resource/macros.xacro (robot description, xacro)
@@ -82,3 +82,125 @@
         <mesh filename="$(find ezrassor_arm_v2)/meshes/platform.dae" scale="2 2 2"></mesh>
     </xacro:macro>
+    <xacro:macro name="ros2_control_arm_joint1">
+        <ros2_control name="GazeboSystem" type="system">
+            <hardware>
+                <plugin>gazebo_ros2_control/GazeboSystem</plugin>
+            </hardware>
+            <joint name="joint1">
+                <command_interface name="position">
+                    <param name="min">-15</param>
+                    <param name="max">15</param>
+                </command_interface>
+                <state_interface name="position">
+                    <param name="initial_value">1.0</param>
+                </state_interface>
+                <state_interface name="velocity"/>
+                <state_interface name="effort"/>
+            </joint>
+        </ros2_control>
+    </xacro:macro>
+    <xacro:macro name="ros2_control_arm_joint2">
+        <ros2_control name="GazeboSystem" type="system">
+            <hardware>
+                <plugin>gazebo_ros2_control/GazeboSystem</plugin>
+            </hardware>
+            <joint name="joint2">
+                <command_interface name="position">
+                    <param name="min">-15</param>
+                    <param name="max">15</param>
+                </command_interface>
+                <state_interface name="position">
+                    <param name="initial_value">1.0</param>
+                </state_interface>
+                <state_interface name="velocity"/>
+                <state_interface name="effort"/>
+            </joint>
+        </ros2_control>
+    </xacro:macro>
+    <xacro:macro name="ros2_control_arm_joint3">
+        <ros2_control name="GazeboSystem" type="system">
+            <hardware>
+                <plugin>gazebo_ros2_control/GazeboSystem</plugin>
+            </hardware>
+            <joint name="joint3">
+                <command_interface name="position">
+                    <param name="min">-15</param>
+                    <param name="max">15</param>
+                </command_interface>
+                <state_interface name="position">
+                    <param name="initial_value">1.0</param>
+                </state_interface>
+                <state_interface name="velocity"/>
+                <state_interface name="effort"/>
+            </joint>
+        </ros2_control>
+    </xacro:macro>
+    <xacro:macro name="ros2_control_arm_joint4">
+        <ros2_control name="GazeboSystem" type="system">
+            <hardware>
+                <plugin>gazebo_ros2_control/GazeboSystem</plugin>
+            </hardware>
+            <joint name="joint4">
+                <command_interface name="position">
+                    <param name="min">-15</param>
+                    <param name="max">15</param>
+                </command_interface>
+                <state_interface name="position">
+                    <param name="initial_value">1.0</param>
+                </state_interface>
+                <state_interface name="velocity"/>
+                <state_interface name="effort"/>
+            </joint>
+        </ros2_control>
+    </xacro:macro>
+    <xacro:macro name="ros2_control_arm_joint5">
+        <ros2_control name="GazeboSystem" type="system">
+            <hardware>
+                <plugin>gazebo_ros2_control/GazeboSystem</plugin>
+            </hardware>
+            <joint name="joint5">
+                <command_interface name="position">
+                    <param name="min">-15</param>
+                    <param name="max">15</param>
+                </command_interface>
+                <state_interface name="position">
+                    <param name="initial_value">1.0</param>
+                </state_interface>
+                <state_interface name="velocity"/>
+                <state_interface name="effort"/>
+            </joint>
+        </ros2_control>
+    </xacro:macro>
+    <xacro:macro name="ros2_control_arm_grabber1">
+        <ros2_control name="GazeboSystem" type="system">
+            <hardware>
+                <plugin>gazebo_ros2_control/GazeboSystem</plugin>
+            </hardware>
+            <joint name="grabber1">
+                <command_interface name="effort">
+                    <param name="min">-1000</param>
+                    <param name="max">1000</param>
+                </command_interface>
+                <state_interface name="position"/>
+                <state_interface name="velocity"/>
+                <state_interface name="effort"/>
+            </joint>
+        </ros2_control>
+    </xacro:macro>
+    <xacro:macro name="ros2_control_arm_grabber2">
+        <ros2_control name="GazeboSystem" type="system">
+            <hardware>
+                <plugin>gazebo_ros2_control/GazeboSystem</plugin>
+            </hardware>
+            <joint name="grabber2">
+                <command_interface name="effort">
+                    <param name="min">-1000</param>
+                    <param name="max">1000</param>
+                </command_interface>
+                <state_interface name="position"/>
+                <state_interface name="velocity"/>
+                <state_interface name="effort"/>
+            </joint>
+        </ros2_control>
+    </xacro:macro>
 </robot>

Commit message: Attempts to fix arm issues caused by ros2_control

File: ezrassor_arm_v2/resource/ezrassor_arm_v2.xacro (robot description, xacro)
@@ -609,5 +609,4 @@
     </actuator>
   </transmission>
-  -->
   <!-- Front Camera Added -->
   <link name="depth_camera_front">
@@ -743,5 +742,5 @@
     <parent link="link1"/>
     <axis xyz="0 0 1" rpy="0 0 0"/>
-    <joint_properties damping="0.0" friction="0.0"/>
+    <joint_properties damping="21.0" friction="10.0"/>
   </joint>
   <joint type="continuous" name="joint2">
@@ -750,5 +749,5 @@
     <parent link="link2"/>
     <axis xyz="0 1 0" rpy="0 0 0"/>
-    <joint_properties damping="0.0" friction="0.0"/>
+    <joint_properties damping="21.0" friction="10.0"/>
   </joint>
   <joint type="continuous" name="joint3">
@@ -757,5 +756,5 @@
     <parent link="link3"/>
     <axis xyz="0 1 0" rpy="0 0 0"/>
-    <joint_properties damping="0.0" friction="0.0"/>
+    <joint_properties damping="21.0" friction="10.0"/>
   </joint>
   <joint type="continuous" name="joint4">
@@ -764,5 +763,5 @@
     <parent link="link4"/>
     <axis xyz="0 1 0" rpy="0 0 0"/>
-    <joint_properties damping="0.0" friction="0.0"/>
+    <joint_properties damping="21.0" friction="10.0"/>
   </joint>
   <joint type="continuous" name="joint5">
@@ -771,5 +770,5 @@
     <parent link="link5"/>
     <axis xyz="0 0 1" rpy="0 0 0"/>
-    <joint_properties damping="0.0" friction="0.0"/>
+    <joint_properties damping="21.0" friction="10.0"/>
   </joint>
   <joint name="arm_camera_joint" type="fixed">
@@ -812,8 +811,10 @@
                 </command_interface>
                 <state_interface name="position">
-                    <param name="initial_value">0.0</param>
+                    <param name="initial_value">1.0</param>
                 </state_interface>
                 <state_interface name="velocity"/>
-                <state_interface name="effort"/>
+                <state_interface name="effort">
+                    <param name='inital_value'>5.0</param>
+                </state_interface>
             </joint>
             <joint name="joint2">
@@ -823,8 +824,10 @@
                 </command_interface>
                 <state_interface name="position">
-                    <param name="initial_value">0.0</param>
+                    <param name="initial_value">1.0</param>
                 </state_interface>
                 <state_interface name="velocity"/>
-                <state_interface name="effort"/>
+                <state_interface name="effort">
+                    <param name='inital_value'>5.0</param>
+                </state_interface>
             </joint>
             <joint name="joint3">
@@ -834,8 +837,10 @@
                 </command_interface>
                 <state_interface name="position">
-                    <param name="initial_value">0.0</param>
+                    <param name="initial_value">1.0</param>
                 </state_interface>
                 <state_interface name="velocity"/>
-                <state_interface name="effort"/>
+                <state_interface name="effort">
+                    <param name='inital_value'>5.0</param>
+                </state_interface>
             </joint>
             <joint name="joint4">
@@ -845,8 +850,10 @@
                 </command_interface>
                 <state_interface name="position">
-                    <param name="initial_value">0.0</param>
+                    <param name="initial_value">1.0</param>
                 </state_interface>
                 <state_interface name="velocity"/>
-                <state_interface name="effort"/>
+                <state_interface name="effort">
+                    <param name='inital_value'>5.0</param>
+                </state_interface>
             </joint>
             <joint name="joint5">
@@ -856,8 +863,10 @@
                 </command_interface>
                 <state_interface name="position">
-                    <param name="initial_value">0.0</param>
+                    <param name="initial_value">1.0</param>
                 </state_interface>
                 <state_interface name="velocity"/>
-                <state_interface name="effort"/>
+                <state_interface name="effort">
+                    <param name='inital_value'>5.0</param>
+                </state_interface>
             </joint>
             <joint name="grabber_joint1">

File: ezrassor_arm_v2/resource/macros.xacro (robot description, xacro)
@@ -82,125 +82,3 @@
         <mesh filename="$(find ezrassor_arm_v2)/meshes/platform.dae" scale="2 2 2"></mesh>
     </xacro:macro>
-    <xacro:macro name="ros2_control_arm_joint1">
-        <ros2_control name="GazeboSystem" type="system">
-            <hardware>
-                <plugin>gazebo_ros2_control/GazeboSystem</plugin>
-            </hardware>
-            <joint name="joint1">
-                <command_interface name="position">
-                    <param name="min">-15</param>
-                    <param name="max">15</param>
-                </command_interface>
-                <state_interface name="position">
-                    <param name="initial_value">1.0</param>
-                </state_interface>
-                <state_interface name="velocity"/>
-                <state_interface name="effort"/>
-            </joint>
-        </ros2_control>
-    </xacro:macro>
-    <xacro:macro name="ros2_control_arm_joint2">
-        <ros2_control name="GazeboSystem" type="system">
-            <hardware>
-                <plugin>gazebo_ros2_control/GazeboSystem</plugin>
-            </hardware>
-            <joint name="joint2">
-                <command_interface name="position">
-                    <param name="min">-15</param>
-                    <param name="max">15</param>
-                </command_interface>
-                <state_interface name="position">
-                    <param name="initial_value">1.0</param>
-                </state_interface>
-                <state_interface name="velocity"/>
-                <state_interface name="effort"/>
-            </joint>
-        </ros2_control>
-    </xacro:macro>
-    <xacro:macro name="ros2_control_arm_joint3">
-        <ros2_control name="GazeboSystem" type="system">
-            <hardware>
-                <plugin>gazebo_ros2_control/GazeboSystem</plugin>
-            </hardware>
-            <joint name="joint3">
-                <command_interface name="position">
-                    <param name="min">-15</param>
-                    <param name="max">15</param>
-                </command_interface>
-                <state_interface name="position">
-                    <param name="initial_value">1.0</param>
-                </state_interface>
-                <state_interface name="velocity"/>
-                <state_interface name="effort"/>
-            </joint>
-        </ros2_control>
-    </xacro:macro>
-    <xacro:macro name="ros2_control_arm_joint4">
-        <ros2_control name="GazeboSystem" type="system">
-            <hardware>
-                <plugin>gazebo_ros2_control/GazeboSystem</plugin>
-            </hardware>
-            <joint name="joint4">
-                <command_interface name="position">
-                    <param name="min">-15</param>
-                    <param name="max">15</param>
-                </command_interface>
-                <state_interface name="position">
-                    <param name="initial_value">1.0</param>
-                </state_interface>
-                <state_interface name="velocity"/>
-                <state_interface name="effort"/>
-            </joint>
-        </ros2_control>
-    </xacro:macro>
-    <xacro:macro name="ros2_control_arm_joint5">
-        <ros2_control name="GazeboSystem" type="system">
-            <hardware>
-                <plugin>gazebo_ros2_control/GazeboSystem</plugin>
-            </hardware>
-            <joint name="joint5">
-                <command_interface name="position">
-                    <param name="min">-15</param>
-                    <param name="max">15</param>
-                </command_interface>
-                <state_interface name="position">
-                    <param name="initial_value">1.0</param>
-                </state_interface>
-                <state_interface name="velocity"/>
-                <state_interface name="effort"/>
-            </joint>
-        </ros2_control>
-    </xacro:macro>
-    <xacro:macro name="ros2_control_arm_grabber1">
-        <ros2_control name="GazeboSystem" type="system">
-            <hardware>
-                <plugin>gazebo_ros2_control/GazeboSystem</plugin>
-            </hardware>
-            <joint name="grabber1">
-                <command_interface name="effort">
-                    <param name="min">-1000</param>
-                    <param name="max">1000</param>
-                </command_interface>
-                <state_interface name="position"/>
-                <state_interface name="velocity"/>
-                <state_interface name="effort"/>
-            </joint>
-        </ros2_control>
-    </xacro:macro>
-    <xacro:macro name="ros2_control_arm_grabber2">
-        <ros2_control name="GazeboSystem" type="system">
-            <hardware>
-                <plugin>gazebo_ros2_control/GazeboSystem</plugin>
-            </hardware>
-            <joint name="grabber2">
-                <command_interface name="effort">
-                    <param name="min">-1000</param>
-                    <param name="max">1000</param>
-                </command_interface>
-                <state_interface name="position"/>
-                <state_interface name="velocity"/>
-                <state_interface name="effort"/>
-            </joint>
-        </ros2_control>
-    </xacro:macro>
 </robot>
